Commit message: style: adding write-up

File: my_bot/urdf/my_bot.xacro (robot description, xacro)
@@ -172,5 +172,5 @@
   </joint>
   <joint type="fixed" name="camera_joint">
-    <origin xyz="0.15 0 0.01" rpy="0 0 0"/>
+    <origin xyz="0.2 0 0.01" rpy="0 0 0"/>
     <child link="camera"/>
     <parent link="chassis"/>
